File: bongoriannes.sch (KiCad schematic (older format))
At the start: 67 parts, among them J1 VRAM, J10 Conn_01x02, J11 Conn_01x02, J12 EXT, J13 Conn_01x02, J14 Conn_01x02, J2 CART_FRONT, J3 CART_BOTTOM, J4 CPU_RP2A03, J5 PRG_WRAM, J6 P1, J7 PPU, J8 P2, J9 Conn_01x02, Q1 2SC2021, Q2 2SC2021, Q3 2SA937, SW1 SW_Push, U1 74LS373, U2 74LS139, U3 74LS368, U4 74LS368, Y1 21.47727

Commit message: clean
Parts:
- removed C1, C10: 51p, Capacitors_SMD:C_0603_HandSoldering, symbol C
- removed C11, C13, C18, C20, C3: 0.1u, Capacitors_THT:C_Disc_D4.3mm_W1.9mm_P5.00mm, symbol C
- removed C12, C9: 68p, Capacitors_SMD:C_0603_HandSoldering, symbol C
- removed C14, C17: 0.1u, Capacitors_SMD:C_0603_HandSoldering, symbol C
- removed C15: 30p, Capacitors_SMD:C_0603_HandSoldering, symbol C
- removed C16: 330p, Capacitors_SMD:C_0603_HandSoldering, symbol C
- removed C19: 1u, Capacitors_SMD:CP_Elec_5x5.3, symbol CP1
- removed C2: 5p, Capacitors_SMD:C_0603_HandSoldering, symbol C
- removed C4: 0.47u, Capacitors_SMD:CP_Elec_5x5.3, symbol CP1
- removed C5: 18p, Capacitors_SMD:C_0603_HandSoldering, symbol C
- removed C6: 30p, SamacSys_Parts:TZ03(B), symbol CTRIM
- removed C7: 220p, Capacitors_SMD:C_0603_HandSoldering, symbol C
- removed C8: 15p, Capacitors_SMD:C_0603_HandSoldering, symbol C
- removed D1: 1S953, Diodes_SMD:D_SOD-123, symbol D
- removed J1: VRAM, Housings_SOIC:SOIC-24W_7.5x15.4mm_Pitch1.27mm, symbol Conn_02x12_Counter_Clockwise
- removed J10, J11, J13, J14, J9: Conn_01x02, Pin_Headers:Pin_Header_Straight_1x02_Pitch2.54mm, symbol Conn_01x02
- removed J12: EXT, Connectors_JST:JST_PH_S15B-PH-K_15x2.00mm_Angled, symbol Conn_01x15
- removed J2: CART_FRONT, Pin_Headers:Pin_Header_Straight_1x30_Pitch2.54mm, symbol Conn_01x30
- removed J3: CART_BOTTOM, Pin_Headers:Pin_Header_Straight_1x30_Pitch2.54mm, symbol Conn_01x30
- removed J4: CPU_RP2A03, Housings_DIP:DIP-40_W15.24mm_Socket_LongPads, symbol Conn_02x20_Counter_Clockwise
- removed J5: PRG_WRAM, Housings_SOIC:SOIC-24W_7.5x15.4mm_Pitch1.27mm, symbol Conn_02x12_Counter_Clockwise
- removed J6: P1, Connectors_JST:JST_PH_S5B-PH-K_05x2.00mm_Angled, symbol Conn_01x05
- removed J7: PPU, Housings_DIP:DIP-40_W15.24mm_Socket_LongPads, symbol Conn_02x20_Counter_Clockwise
- removed J8: P2, Connectors_JST:JST_PH_S6B-PH-K_06x2.00mm_Angled, symbol Conn_01x06
- removed JP1: Jumper, Capacitors_SMD:C_0603_HandSoldering, symbol Jumper
- removed JP15: PD0, Pin_Headers:Pin_Header_Straight_1x02_Pitch1.27mm, symbol Jumper_NO_Small
- removed JP17: PD1, Pin_Headers:Pin_Header_Straight_1x02_Pitch1.27mm, symbol Jumper_NO_Small
- removed JP18: PD7, Pin_Headers:Pin_Header_Straight_1x02_Pitch1.27mm, symbol Jumper_NO_Small
- removed JP19: PD2, Pin_Headers:Pin_Header_Straight_1x02_Pitch1.27mm, symbol Jumper_NO_Small
- removed JP20: PD6, Pin_Headers:Pin_Header_Straight_1x02_Pitch1.27mm, symbol Jumper_NO_Small
- removed JP21: PD3, Pin_Headers:Pin_Header_Straight_1x02_Pitch1.27mm, symbol Jumper_NO_Small
- removed JP22: PD5, Pin_Headers:Pin_Header_Straight_1x02_Pitch1.27mm, symbol Jumper_NO_Small
- removed JP23: PD4, Pin_Headers:Pin_Header_Straight_1x02_Pitch1.27mm, symbol Jumper_NO_Small
- removed Q1, Q2: 2SC2021, Pin_Headers:Pin_Header_Straight_1x03_Pitch2.54mm, symbol 2SC1815
- removed Q3: 2SA937, Pin_Headers:Pin_Header_Straight_1x03_Pitch2.54mm, symbol 2SA1015
- removed R1, R4, R5: 1.2k, Resistors_SMD:R_0603_HandSoldering, symbol R
- removed R10: 20k, Resistors_SMD:R_0603_HandSoldering, symbol R
- removed R11, R14: 100, Resistors_SMD:R_0603_HandSoldering, symbol R
- removed R12: 100k, Resistors_SMD:R_0603_HandSoldering, symbol R
- removed R13: 12k, Resistors_SMD:R_0603_HandSoldering, symbol R
- removed R2: 220k, Resistors_SMD:R_0603_HandSoldering, symbol R
- removed R3: 150k, Resistors_SMD:R_0603_HandSoldering, symbol R
- removed R6: 220, Resistors_SMD:R_0603_HandSoldering, symbol R
- removed R7: 2.2k, Resistors_SMD:R_0603_HandSoldering, symbol R
- removed R8, R9: 10k, Resistors_SMD:R_0603_HandSoldering, symbol R
- removed SW1: SW_Push, Pin_Headers:Pin_Header_Straight_1x02_Pitch2.54mm, symbol SW_Push
- removed U1: 74LS373, Housings_SOIC:SO-20_12.8x7.5mm_Pitch1.27mm, symbol 74LS373
- removed U2: 74LS139, Housings_SSOP:SOP-16_4.4x10.4mm_Pitch1.27mm, symbol 74LS139
- removed U3, U4: 74LS368, Housings_SSOP:SOP-16_4.4x10.4mm_Pitch1.27mm, symbol 74LS368
- removed Y1: 21.47727, Crystals:Crystal_HC49-U_Vertical, symbol Crystal
Connections:
- no-connect marks 4 -> 0

Commit message: meishi_size
Parts:
- added C1, C2, C3, C4, C5, C6, C7, C8, C9: 0.1u, Capacitor_SMD:C_0805_2012Metric_Pad1.15x1.40mm_HandSolder, symbol Device:C
- added C10: 330p, Capacitor_THT:C_Disc_D3.0mm_W1.6mm_P2.50mm, symbol Device:C
- added C11: 30p, Capacitor_THT:C_Disc_D3.0mm_W1.6mm_P2.50mm, symbol Device:C
- added C12, C21: 68p, Capacitor_THT:C_Disc_D3.0mm_W1.6mm_P2.50mm, symbol Device:C
- added C13: 0.47u, Capacitor_THT:CP_Radial_D5.0mm_P2.00mm, symbol Device:CP1
- added C14, C15, C17, C19: 0.1u, Capacitor_THT:C_Disc_D3.0mm_W1.6mm_P2.50mm, symbol Device:C
- added C16: 220u, Capacitor_THT:CP_Radial_D8.0mm_P3.50mm, symbol Device:CP
- added C18: 1u, Capacitor_THT:CP_Radial_D5.0mm_P2.00mm, symbol Device:CP
- added C20: 4.7u, Capacitor_THT:CP_Radial_D5.0mm_P2.00mm, symbol Device:CP
- added CX1: 22p, Capacitor_THT:C_Disc_D3.0mm_W1.6mm_P2.50mm, symbol Device:C
- added CX2: 15p, Capacitor_THT:C_Disc_D3.0mm_W1.6mm_P2.50mm, symbol Device:C
- added CX3: CTRIM, Capacitor_SMD:C_Trimmer_Murata_TZC3, symbol Device:CTRIM
- added D1: 1S953, bongorian:DIODE_SHORT, symbol Device:D
- added D2: LED, LED_THT:LED_D3.0mm, symbol Device:LED
- added EXT1: 1-10, Connector_PinHeader_1.27mm:PinHeader_2x10_P1.27mm_Vertical_SMD, symbol Connector_Generic:Conn_02x10_Odd_Even
- added EXT2: 11-20, Connector_PinHeader_1.27mm:PinHeader_2x10_P1.27mm_Vertical_SMD, symbol Connector_Generic:Conn_02x10_Odd_Even
- added EXT3: 21-30, Connector_PinHeader_1.27mm:PinHeader_2x10_P1.27mm_Vertical_SMD, symbol Connector_Generic:Conn_02x10_Odd_Even
- added J1: P1, Connector_PinHeader_2.54mm:PinHeader_1x05_P2.54mm_Vertical, symbol Connector:Conn_01x05_Male
- added J2: P2, Connector_PinHeader_2.54mm:PinHeader_1x06_P2.54mm_Vertical, symbol Connector:Conn_01x06_Male
- added J3: P3, Connector_PinHeader_1.00mm:PinHeader_1x15_P1.00mm_Vertical, symbol Connector:Conn_01x15_Male
- added J4: VIDEO, bongorian:RCA_RJ2410N, symbol Connector:Conn_Coaxial
- added J5: AUDIO, bongorian:RCA_RJ2410N, symbol Connector:Conn_Coaxial
- added JP1: CLOCK, Jumper:SolderJumper-3_P1.3mm_Open_RoundedPad1.0x1.5mm, symbol Jumper:Jumper_3_Open
- added Q1: 2SA1015, Package_TO_SOT_THT:TO-92_Inline, symbol bongoriannes-rescue:2SA1015
- added R1: 1.2k, Resistor_THT:R_Axial_DIN0204_L3.6mm_D1.6mm_P5.08mm_Horizontal, symbol Device:R
- added R10: 100k, Resistor_THT:R_Axial_DIN0204_L3.6mm_D1.6mm_P5.08mm_Horizontal, symbol Device:R
- added R11: 12k, Resistor_THT:R_Axial_DIN0204_L3.6mm_D1.6mm_P5.08mm_Horizontal, symbol Device:R
- added R12, R8: 100, Resistor_THT:R_Axial_DIN0204_L3.6mm_D1.6mm_P5.08mm_Horizontal, symbol Device:R
- added R13: 1k, Resistor_THT:R_Axial_DIN0204_L3.6mm_D1.6mm_P5.08mm_Horizontal, symbol Device:R
- added R2: 1M, Resistor_THT:R_Axial_DIN0204_L3.6mm_D1.6mm_P5.08mm_Horizontal, symbol Device:R
- added R3: R, Resistor_THT:R_Axial_DIN0204_L3.6mm_D1.6mm_P5.08mm_Horizontal, symbol Device:R
- added R4: 150, Resistor_THT:R_Axial_DIN0204_L3.6mm_D1.6mm_P5.08mm_Horizontal, symbol Device:R
- added R5: 75, Resistor_THT:R_Axial_DIN0204_L3.6mm_D1.6mm_P5.08mm_Horizontal, symbol Device:R
- added R6, R9: 10k, Resistor_THT:R_Axial_DIN0204_L3.6mm_D1.6mm_P5.08mm_Horizontal, symbol Device:R
- added R7: 20k, Resistor_THT:R_Axial_DIN0204_L3.6mm_D1.6mm_P5.08mm_Horizontal, symbol Device:R
- added RN1, RN2, RN3: MNR04MRAPJ103, bongorian:RESCAX50P100X200X36-8N, symbol SamacSys_Parts:MNR04MRAPJ103
- added SW1: SW_Push, keyswitches:PG1350, symbol bongoriannes-rescue:SW_Push
- added U1: 2A03_CPU, bongorian:DIP-40_W15.24mm_LongPads_hoso, symbol Connector_Generic:Conn_02x20_Counter_Clockwise
- added U2: 2C02_PPU, bongorian:DIP-40_W15.24mm_LongPads_hoso, symbol Connector_Generic:Conn_02x20_Counter_Clockwise
- added U3: SRAM, Package_SO:SOIC-24W_7.5x15.4mm_P1.27mm, symbol Connector_Generic:Conn_02x12_Counter_Clockwise
- added U4: VRAM, Package_SO:SOIC-24W_7.5x15.4mm_P1.27mm, symbol Connector_Generic:Conn_02x12_Counter_Clockwise
- added U5: 74LS373, Package_SO:SOIC-20W_7.5x12.8mm_P1.27mm, symbol 74xx:74LS373
- added U6: 74LS139, Package_SO:SOIC-16_3.9x9.9mm_P1.27mm, symbol 74xx:74LS139
- added U7, U8: 74LS368, Package_SO:SOIC-16_3.9x9.9mm_P1.27mm, symbol 74xx:74LS368
- added U9: 74HC04, Package_SO:SOIC-14_3.9x8.7mm_P1.27mm, symbol 74xx:74HC04
- added Y1: Crystal, Crystal:Crystal_HC49-4H_Vertical, symbol Device:Crystal
Connections:
- new net: C12.1, D1.1 (K), R1.2, U3.18 (Pin_18)
- new net: U6.1 (E), U6.11 (O1)
- new net: CX1.1, R2.2, U9.1, Y1.1
- new net: CX2.1, CX3.1, R2.1, U9.2, U9.3, Y1.2
- new net: U9.11, U9.13, U9.4, U9.5, U9.9
- new net: JP1.2 (C), U9.10, U9.12, U9.6, U9.8
- new net: D2.1 (K), R3.1
- new net: C16.1, Q1.1 (E), R4.2
- new net: C16.2, R5.2
- new net: J4.1 (In), R5.1
- new net: C18.2, R11.2, R7.2, R9.2
- new net: J5.1 (In), R13.1
- new net: C20.2, R13.2
- new net 4016_CUP$: J1.4 (Pin_4), J3.14 (Pin_14), RN1.6, U8.7 (O3a)
- new net 4016_D0$: J1.2 (Pin_2), RN1.7, U8.2 (I1)
- new net 4016_D1$: J3.13 (Pin_13), RN1.8, U8.4 (I2)
- new net 4017_CUP$: J2.5 (Pin_5), J3.9 (Pin_9), RN2.6, U7.3 (O1a)
- new net 4017_D0$: J2.3 (Pin_3), J3.8 (Pin_8), RN2.7, U7.14 (I6)
- new net 4017_D1$: J3.7 (Pin_7), RN2.8, U7.4 (I2)
- new net 4017_D2$: J3.6 (Pin_6), RN3.5, U7.12 (I5)
- new net 4017_D3$: J3.5 (Pin_5), RN3.6, U7.6 (I3)
- new net 4017_D4$: J3.4 (Pin_4), RN3.7, U7.10 (I4)
- new net A0: EXT2.5 (Pin_5), U1.4 (Pin_4), U2.12 (Pin_12), U3.8 (Pin_8)
- new net A1: EXT2.3 (Pin_3), U1.5 (Pin_5), U2.11 (Pin_11), U3.7 (Pin_7)
- new net A10: EXT1.5 (Pin_5), U1.14 (Pin_14), U3.19 (Pin_19)
- new net A11: EXT1.3 (Pin_3), U1.15 (Pin_15)
- new net A12: EXT1.6 (Pin_6), U1.16 (Pin_16)
- new net A13: EXT1.8 (Pin_8), U1.17 (Pin_17), U6.2 (A0)
- new net A14: EXT1.10 (Pin_10), U1.18 (Pin_18), U6.3 (A1)
- new net A15: U1.19 (Pin_19), U6.13 (A1)
- new net A2: EXT2.1 (Pin_1), U1.6 (Pin_6), U2.10 (Pin_10), U3.6 (Pin_6)
- new net A3: EXT1.19 (Pin_19), U1.7 (Pin_7), U3.5 (Pin_5)
- new net A4: EXT1.17 (Pin_17), U1.8 (Pin_8), U3.4 (Pin_4)
- new net A5: EXT1.15 (Pin_15), U1.9 (Pin_9), U3.3 (Pin_3)
- new net A6: EXT1.13 (Pin_13), U1.10 (Pin_10), U3.2 (Pin_2)
- new net A7: EXT1.11 (Pin_11), U1.11 (Pin_11), U3.1 (Pin_1)
- new net A8: EXT1.9 (Pin_9), U1.12 (Pin_12), U3.23 (Pin_23)
- new net A9: EXT1.7 (Pin_7), U1.13 (Pin_13), U3.22 (Pin_22)
- new net ALE$%: U2.39 (Pin_39), U5.11 (LE)
- new net AUX_A: R7.1, R8.2, U1.1 (Pin_1)
- new net AUX_B: R11.1, R12.2, U1.2 (Pin_2)
- new net CLKOUT: EXT1.4 (Pin_4), U1.31 (Pin_31), U6.14 (A0), U7.2 (I1), U8.6 (I3)
- new net CPU_CLK: JP1.3 (B), U1.29 (Pin_29)
- new net D0: EXT2.6 (Pin_6), U1.28 (Pin_28), U2.2 (Pin_2), U3.9 (Pin_9), U7.13 (O6b), U8.3 (O1a)
- new net D1: EXT2.4 (Pin_4), U1.27 (Pin_27), U2.3 (Pin_3), U3.10 (Pin_10), U7.5 (O2a), U8.5 (O2a)
- new net D2: EXT2.2 (Pin_2), U1.26 (Pin_26), U2.4 (Pin_4), U3.11 (Pin_11), U7.11 (O5b), U8.9 (O4a)
- new net D3: EXT1.20 (Pin_20), U1.25 (Pin_25), U2.5 (Pin_5), U3.13 (Pin_13), U7.7 (O3a)
- new net D4: EXT1.18 (Pin_18), U1.24 (Pin_24), U2.6 (Pin_6), U3.14 (Pin_14), U7.9 (O4a)
- new net D5: EXT1.16 (Pin_16), U1.23 (Pin_23), U2.7 (Pin_7), U3.15 (Pin_15)
- new net D6: EXT1.14 (Pin_14), U1.22 (Pin_22), U2.8 (Pin_8), U3.16 (Pin_16)
- new net D7: EXT1.12 (Pin_12), U1.21 (Pin_21), U2.9 (Pin_9), U3.17 (Pin_17)
- new net DBE#: C10.1, C11.1, U2.13 (Pin_13), U6.5 (O1)
- new net GND: C1.2, C10.2, C11.2, C12.2, C13.2, C14.1, C15.1, C17.2, C19.2, C2.2, C21.2, C3.2, C4.2, C5.2, C6.2, C7.2, C8.2, C9.2, CX1.2, CX2.2, CX3.2, EXT1.1 (Pin_1), EXT2.11 (Pin_11), J1.1 (Pin_1), J2.2 (Pin_2), J3.1 (Pin_1), J4.2 (Ext), J5.2 (Ext), Q1.2 (C), R12.1, R3.2, R8.1, SW1.2, U1.20 (Pin_20), U1.30 (Pin_30), U2.14 (Pin_14), U2.15 (Pin_15), U2.16 (Pin_16), U2.17 (Pin_17), U2.20 (Pin_20), U3.12 (Pin_12), U3.20 (Pin_20), U4.12 (Pin_12), U5.1 (OE), U5.10 (GND), U6.15 (E), U6.8 (GND), U7.8 (GND), U8.15 (OEb), U8.8 (GND), U9.7 (GND)
- new net INP0#: U1.36 (Pin_36), U8.1 (OEa)
- new net INP1#: U1.35 (Pin_35), U7.1 (OEa), U7.15 (OEb)
- new net IRQ#$: EXT2.9 (Pin_9), J3.3 (Pin_3), RN2.5, U1.32 (Pin_32)
- new net MIC_IN: J2.1 (Pin_1), R6.2, R9.1
- new net MIC_IN': C17.1, R6.1, U8.10 (I4)
- new net NMI#$: RN3.8, U1.33 (Pin_33), U2.19 (Pin_19)
- new net OUT0: J1.3 (Pin_3), J2.4 (Pin_4), J3.12 (Pin_12), U1.39 (Pin_39)
- new net OUT1: J3.11 (Pin_11), U1.38 (Pin_38)
- new net OUT2: J3.10 (Pin_10), U1.37 (Pin_37)
- new net PA0: EXT3.9 (Pin_9), U4.8 (Pin_8), U5.19 (O7)
- new net PA1: EXT3.7 (Pin_7), U4.7 (Pin_7), U5.16 (O6)
- new net PA10$%: EXT3.6 (Pin_6), U2.28 (Pin_28)
- new net PA11$%: EXT3.8 (Pin_8), U2.27 (Pin_27)
- new net PA12$%: EXT3.10 (Pin_10), U2.26 (Pin_26)
- new net PA13$%: EXT3.12 (Pin_12), U2.25 (Pin_25), U8.12 (I5)
- new net PA13': EXT2.18 (Pin_18), U8.11 (O5b)
- new net PA2: EXT3.5 (Pin_5), U4.6 (Pin_6), U5.15 (O5)
- new net PA3: EXT3.3 (Pin_3), U4.5 (Pin_5), U5.12 (O4)
- new net PA4: EXT3.1 (Pin_1), U4.4 (Pin_4), U5.9 (O3)
- new net PA5: EXT2.19 (Pin_19), U4.3 (Pin_3), U5.6 (O2)
- new net PA6: EXT2.17 (Pin_17), U4.2 (Pin_2), U5.5 (O1)
- new net PA7: EXT2.20 (Pin_20), U4.1 (Pin_1), U5.2 (O0)
- new net PA8$%: EXT3.2 (Pin_2), U2.30 (Pin_30), U4.23 (Pin_23)
- new net PA9$%: EXT3.4 (Pin_4), U2.29 (Pin_29), U4.22 (Pin_22)
- new net PD0: EXT3.17 (Pin_17), U2.38 (Pin_38), U4.9 (Pin_9), U5.18 (D7)
- new net PD1: EXT3.15 (Pin_15), U2.37 (Pin_37), U4.10 (Pin_10), U5.17 (D6)
- new net PD2: EXT3.13 (Pin_13), U2.36 (Pin_36), U4.11 (Pin_11), U5.14 (D5)
- new net PD3: EXT3.11 (Pin_11), U2.35 (Pin_35), U4.13 (Pin_13), U5.13 (D4)
- new net PD4: EXT3.20 (Pin_20), U2.34 (Pin_34), U4.14 (Pin_14), U5.8 (D3)
- new net PD5: EXT3.18 (Pin_18), U2.33 (Pin_33), U4.15 (Pin_15), U5.7 (D2)
- new net PD6: EXT3.16 (Pin_16), U2.32 (Pin_32), U4.16 (Pin_16), U5.4 (D1)
- new net PD7: EXT3.14 (Pin_14), U2.31 (Pin_31), U4.17 (Pin_17), U5.3 (D0)
- new net PPU_CLK: JP1.1 (A), U2.18 (Pin_18)
- new net RAMSEL#: D1.2 (A), R1.1, U6.4 (O0)
- new net RD#$%: C21.1, EXT2.13 (Pin_13), U2.24 (Pin_24), U4.20 (Pin_20)
- new net RES#$%: C13.1, SW1.1, U1.3 (Pin_3)
- new net ROMSEL#: EXT2.8 (Pin_8), U6.9 (O3)
- new net R_W#: EXT2.7 (Pin_7), U1.34 (Pin_34), U2.1 (Pin_1), U3.21 (Pin_21)
- new net SOUND_I: C19.1, EXT2.10 (Pin_10), J3.2 (Pin_2), R10.2, U8.13 (O6b)
- new net SOUND_I': C18.1, R10.1, U8.14 (I6)
- new net SOUND_OUT: C20.1, EXT2.12 (Pin_12)
- new net VCC: C1.1, C14.2, C15.2, C2.1, C3.1, C4.1, C5.1, C6.1, C7.1, C8.1, C9.1, D2.2 (A), EXT1.2 (Pin_2), EXT3.19 (Pin_19), J1.5 (Pin_5), J2.6 (Pin_6), J3.15 (Pin_15), R4.1, RN1.1, RN1.2, RN1.3, RN1.4, RN2.1, RN2.2, RN2.3, RN2.4, RN3.1, RN3.2, RN3.3, RN3.4, U1.40 (Pin_40), U2.22 (Pin_22), U2.40 (Pin_40), U3.24 (Pin_24), U4.24 (Pin_24), U5.20 (VCC), U6.16 (VCC), U7.16 (VCC), U8.16 (VCC), U9.14 (VCC)
- new net VIDEO_OUT: Q1.3 (B), U2.21 (Pin_21)
- new net VRAMA10: EXT2.15 (Pin_15), U4.19 (Pin_19)
- new net VRAMCS#: EXT2.16 (Pin_16), U4.18 (Pin_18)
- new net WR#$%: EXT2.14 (Pin_14), U2.23 (Pin_23), U4.21 (Pin_21)
- no-connect marks 0 -> 5
